Commit message: improved order of the lessons and added timeout before spawning the robot in gazebo

File: Section4-Digital_Twin/arduinobot_ws/src/arduinobot_description/urdf/arduinobot.urdf.xacro (robot description, xacro)
@@ -191,23 +191,3 @@
     <xacro:default_transmission number="3"/>
     <xacro:default_transmission number="4"/>
-    <!-- gazebo ros_control plugin -->
-    <gazebo>
-        <plugin name="gazebo_ros_control" filename="libgazebo_ros_control.so">
-            <robotNamespace>/arduinobot</robotNamespace>
-            <robotSimType>gazebo_ros_control/DefaultRobotHWSim</robotSimType>
-            <legacyModeNS>true</legacyModeNS>
-        </plugin>
-    </gazebo>
-    <gazebo>
-      <plugin name="mimic_joint_plugin" filename="libroboticsgroup_gazebo_mimic_joint_plugin.so">
-        <joint>joint_4</joint>
-        <mimicJoint>joint_5</mimicJoint>
-        <hasPID />
-        <multiplier>-1.0</multiplier>
-        <offset>0</offset>
-        <sensitiveness>0.0</sensitiveness>
-        <maxEffort>${effort}</maxEffort>
-        <robotNamespace>/arduinobot</robotNamespace>
-      </plugin>
-    </gazebo>
 </robot>

Commit message: sync section 4 with lessons

File: Section4-Digital_Twin/arduinobot_ws/src/arduinobot_description/urdf/arduinobot.urdf.xacro (robot description, xacro)
@@ -191,3 +191,19 @@
     <xacro:default_transmission number="3"/>
     <xacro:default_transmission number="4"/>
+    <!-- gazebo ros_control plugin -->
+    <gazebo>
+        <plugin name="gazebo_ros_control" filename="libgazebo_ros_control.so">
+            <robotNamespace>/arduinobot</robotNamespace>
+            <robotSimType>gazebo_ros_control/DefaultRobotHWSim</robotSimType>
+            <legacyModeNS>true</legacyModeNS>
+        </plugin>
+        <plugin name="joint_5_mimic_joint_4" filename="libroboticsgroup_gazebo_mimic_joint_plugin.so">
+          <joint>joint_4</joint>
+          <mimicJoint>joint_5</mimicJoint>
+          <multiplier>-1.0</multiplier>
+          <offset>0</offset>
+          <maxEffort>${effort}</maxEffort>
+          <robotNamespace>/arduinobot</robotNamespace>
+        </plugin>
+    </gazebo>
 </robot>
